File: pcb/Leyden_Jar.kicad_pcb (KiCad board)
At the start: 4 copper layers, 85 x 26.5 mm, 90 parts, among them J1 USB_C_Receptacle_USB2.0, J2 Switch matrix connector, J3 SWD_Connector, J4 Ext Conn, SW1 B3U-3000P, SW2 B3U-3000P, U1 W25Q16JVUXIQ, U10 MCP4716A0T-E/CH, U2 LMV339, U3 USBLC6-2SC6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

Commit message: [feature] Revision 3 design delivery.
Parts:
- added SW3: B3U-1000P, Leyden_Jar:SPST_B3U-1000P, F.Cu at (43.2, 1.25)
- added SW4: B3U-1000P, Leyden_Jar:SPST_B3U-1000P, F.Cu at (53.2, 1.25)
- J3: value SWD_Connector -> SWD/I2C; footprint Leyden_Jar:SWD_Header -> Leyden_Jar:PinHeader_2x03_P2.54mm_Horizontal
- SW1, SW2: value B3U-3000P -> B3U-1000P; footprint Leyden_Jar:SPST_B3U-3000P -> Leyden_Jar:SPST_B3U-1000P; moved to B.Cu
- moved H3 1.83 mm to (34.7, 22.7)
- moved J3 0.66 mm to (11.6, 2.30)
Connections:
- J3 pad 2: /SWCLK -> /3V3
- J3 pad 3: /SWIO -> /SWCLK
- J4 pad 5: unconnected-(J4-Pad5) -> /3V3
Routing:
- net /SCL: track 46.0 -> 66.3 mm
- net /SDA: track 47.4 -> 67.5 mm
- net /SWCLK: track 26.2 -> 32.1 mm
- net /SWIO: track 25.6 -> 30.4 mm
- net GND: track 40.1 -> 43.3 mm
- net /USB_BOOT: track 3.87 -> 5.38 mm, vias 0 -> 1
- net /D-: track 13.4 -> 11.9 mm, vias 2 -> 0
- net /RUN: track 16.8 -> 17.9 mm, vias 2 -> 3
- net /D+: track 12.0 -> 12.2 mm, vias 2 -> 0
Other:
- board text added: "Beam Spring and Model F PCB Rev 3"
- board text added: "Boot"
- board text added: "Swd/I2C"
- board text removed: "Beam Spring and Model F PCB Rev 2"
- board text removed: "Bootsel"
- board text removed: "Gnd"
- board text removed: "Swclk"
- board text removed: "Swd"
- board text removed: "Swio"
