File: pcb/Leyden_Jar.kicad_sch (KiCad schematic)
At the start: 90 parts, among them J1 USB_C_Receptacle_USB2.0, J2 Switch matrix connector, J3 SWD_Connector, J4 Ext Conn, SW1 B3U-3000P, SW2 B3U-3000P, U1 W25Q16JVUXIQ, U10 MCP4716A0T-E/CH, U2 LMV339, U3 USBLC6-2SC6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

Commit message: [feature] Revision 3 design delivery.
Parts:
- removed J3: SWD_Connector, Leyden_Jar:SWD_Header, symbol Connector:Conn_01x03_Male
- added J3: SWD/I2C, Leyden_Jar:PinHeader_2x03_P2.54mm_Horizontal, symbol Connector_Generic:Conn_02x03_Odd_Even
- added SW3, SW4: B3U-1000P, Leyden_Jar:SPST_B3U-1000P, symbol Switch:SW_Push
- SW1, SW2: value B3U-3000P -> B3U-1000P; footprint Leyden_Jar:SPST_B3U-3000P -> Leyden_Jar:SPST_B3U-1000P; LCSC C963349 -> C5362268
- U2, U6: LCSC C273648 -> C273648
- U2, U6: LCSC (none) -> C273648; Manufacturer ID (none) -> LMV339; Mouser (none) -> 863-LMV339DTBR2G
Connections:
- net 3V3: now also J4.5 (Pin_5), J3.2 (Pin_2)
- net GND: now also J3.1 (Pin_1), SW3.1, SW4.1
- net RUN: now also SW3.2
- net SCL: now also J3.6 (Pin_6)
- net SDA: now also J3.4 (Pin_4)
- net SWCLK: now also J3.3 (Pin_3)
- net SWIO: now also J3.5 (Pin_5)
- net USB_BOOT: now also SW4.2
- no-connect marks 9 -> 8
Other:
- note added: "SWD/I2C connector"
- note removed: "SWD connector"
- moved on the sheet: R40, SW1, SW2
