File: pcb/ps2_at_daughterboard/ps2_pcb.kicad_pcb (KiCad board)
At the start: 2 copper layers, 35 x 26.5 mm, 18 parts, among them J1 Conn_02x03_Odd_Even, J2 USB_C_Receptacle_USB2.0, Q1 BSS138, Q2 BSS138, U2 MIC2009A-1YM6, U3 USBLC6-2SC6

Commit message: [feature] PS2 daughterboard project conversion to Kicad 10.x
Parts:
- H1: value Val** -> Rico_Logo
- J2: value USB_C_Receptacle_USB2.0 -> USB_C_Receptacle_USB2.0_16P
- Q1, Q2: footprint Model-F:SOT-23 -> Package_TO_SOT_SMD:SOT-23
- U3: footprint Model-F:SOT-23-6 -> Package_TO_SOT_SMD:SOT-23-6

Commit message: [feature] PS2 daughterboard design Rev 2 ready for fabrication.
Parts:
- added D1: D_Schottky_Small, Model-F:D_SOD-123, F.Cu at (47.0, 40.7)
Connections:
- J1 pad 1: OUT_5V -> CONN_5V
Routing:
- net CONN_5V: track 0.00 -> 7.94 mm, vias 0 -> 1
- net OUT_5V: track 40.0 -> 33.1 mm, vias 2 -> 3
Other:
- board text added: "PS2 AT to USB Daughterboard Rev 2"
- board text removed: "PS2 AT to USB Daughterboard Rev 1"
